Commit message: 添加相关参数注释

File: src/rm_nav_bringup/urdf/sentry_robot_real.xacro (robot description, xacro)
@@ -11,6 +11,6 @@
     </inertial>
   </xacro:macro>
-  <!-- base_link to livox_frame -->
-  <xacro:arg name="xyz" default="0.0 0.045 0.49" />
+  <!-- base_link to gimbal_link -->
+  <xacro:arg name="xyz" default="0.0 0.045 0.35" />
   <xacro:arg name="rpy" default="0 0 0" />
   <link name="base_link">
@@ -31,4 +31,22 @@
     </collision>
     <xacro:default_inertial mass="8.2"/>
+  </link>
+  <link name="gimbal_link">
+    <visual>
+      <geometry>
+        <cylinder radius="0.04" length="0.06"/>
+      </geometry>
+      <origin rpy="0 0 0" xyz="0 0 0"/>
+      <material name="silver">
+        <color rgba="0.8 0.8 0.8 1"/>
+      </material>
+    </visual>
+    <collision>
+      <geometry>
+        <cylinder radius="0.04" length="0.06"/>
+      </geometry>
+      <origin rpy="0 0 0" xyz="0 0 0"/>
+    </collision>
+    <xacro:default_inertial mass="0.6"/>
   </link>
   <link name="wheel_1">
@@ -140,7 +158,12 @@
     </visual>
   </link>
-  <joint name="livox_joint" type="fixed">
+  <joint name="base_to_gimbal" type="fixed">
     <origin xyz="$(arg xyz)" rpy="$(arg rpy)" />
     <parent link="base_link"/>
+    <child link="gimbal_link"/>
+  </joint>
+  <joint name="livox_joint" type="fixed">
+    <origin xyz="0 0 0" rpy="0 0 0" />
+    <parent link="gimbal_link"/>
     <child link="livox_frame"/>
   </joint>

File: src/rm_nav_bringup/urdf/sentry_robot_sim.xacro (robot description, xacro)
@@ -11,6 +11,6 @@
     </inertial>
   </xacro:macro>
-  <!-- base_link to livox_frame -->
-  <xacro:arg name="xyz" default="0.12 0.0 0.175" />
+  <!-- base_link to gimbal_link -->
+  <xacro:arg name="xyz" default="0.12 0.0 0.35" />
   <xacro:arg name="rpy" default="0 0 0" />
   <link name="dummy"/>
@@ -33,7 +33,30 @@
     <xacro:default_inertial mass="8.2"/>
   </link>
+  <link name="gimbal_link">
+    <visual>
+      <geometry>
+        <cylinder radius="0.04" length="0.06"/>
+      </geometry>
+      <origin rpy="0 0 0" xyz="0 0 0"/>
+      <material name="silver">
+        <color rgba="0.8 0.8 0.8 1"/>
+      </material>
+    </visual>
+    <collision>
+      <geometry>
+        <cylinder radius="0.04" length="0.06"/>
+      </geometry>
+      <origin rpy="0 0 0" xyz="0 0 0"/>
+    </collision>
+    <xacro:default_inertial mass="0.6"/>
+  </link>
   <joint name="dummy_joint" type="fixed">
      <parent link="dummy"/>
      <child link="base_link"/>
+  </joint>
+  <joint name="base_to_gimbal" type="fixed">
+    <origin xyz="$(arg xyz)" rpy="$(arg rpy)" />
+    <parent link="base_link"/>
+    <child link="gimbal_link"/>
   </joint>
   <link name="wheel_1">
@@ -181,4 +204,7 @@
   <gazebo reference="imu_link">
     <material>Gazebo/BuildingFrame</material>
+  </gazebo>
+  <gazebo reference="gimbal_link">
+    <material>Gazebo/Grey</material>
   </gazebo>
   <gazebo reference="livox_frame">
@@ -229,6 +255,6 @@
   <!-- Livox-Mid360  -->
   <xacro:include filename="$(find ros2_livox_simulation)/urdf/mid360.xacro" />
-  <xacro:mid360 name="livox_frame" parent="base_link" topic="/livox/lidar">
-    <origin xyz="$(arg xyz)" rpy="$(arg rpy)" />
+  <xacro:mid360 name="livox_frame" parent="gimbal_link" topic="/livox/lidar">
+    <origin xyz="0 0 0" rpy="0 0 0" />
   </xacro:mid360>
 </robot>

File: src/rm_robot_description/urdf/sentry.urdf.xacro (robot description, xacro)
@@ -3,12 +3,18 @@
   <!-- Base links -->
   <link name="livox_frame" />
+  <link name="gimbal_link" />
   <link name="base_link" />
   <link name="base_footprint" />
   <!-- Base joints -->
+  <joint name="livox_to_gimbal_joint" type="fixed">
+    <origin xyz="0 0 0" rpy="0 0 0" />
+    <parent link="livox_frame" />
+    <child link="gimbal_link" />
+    <axis xyz="0 0 0" />
+  </joint>
   <joint name="base_joint" type="fixed">
-    <origin xyz="-0.22 -0.11 0.12" rpy="0 0 0" />
-    <parent link="livox_frame" />
+    <parent link="gimbal_link"/>
     <child link="base_link" />
-    <axis xyz="0 0 0" />
+    <origin xyz="-0.22 -0.11 0.12" rpy="0 0 0"/>
   </joint>
   <joint name="base_footprint_joint" type="fixed">
